File: DueFinn.sch (KiCad schematic (older format))
At the start: 59 parts

Commit message: SAM3X power and USB con included
Parts:
- removed L?: SRR0604-100ML, symbol pspice:INDUCTOR
- removed U?: ATSAM3X8EA-AU, DueFinn:QFP50P2200X2200X145-144N, symbol DueFinn:ATSAM3X8EA-AU
- added C?: 47u, symbol Device:CP1
- added C? (x6): 10u, symbol Device:CP1
- added C? (x9): 100n, symbol Device:C
- added C?: 10n, symbol Device:C
- added D?: SS1P3L, symbol Device:D_Schottky
- added F?: Polyfuse, symbol Device:Polyfuse
- added FB? (x4): MH2029-300Y, symbol Device:Ferrite_Bead
- added J?: USB_OTG, symbol Connector:USB_OTG
- added JP?: Jumper_NC_Dual, symbol Device:Jumper_NC_Dual
- added L?: SRR0604-100ML, symbol Device:L
- added R?: 10k, symbol Device:R
- added RV? (x3): CG0603MLC-05E, symbol Device:Varistor
- added U?: ATSAM3X8EA-AU, QFP50P2200X2200X145-144N, symbol DueFinn:ATSAM3X8EA-AU
Connections:
- net labels added: 9V_RAW, D+, D-, UOTGID, USBVCC, VBUS, VDDANA, VDDUTMI
- wire segments 153 -> 248
- no-connect marks 2 -> 3
Other:
- note added: "DIODE!?"
- note added: "Erase"
- note added: "Not Erase"
- moved on the sheet: C?, J?, R?, U?, U?A, U?B

Commit message: Added SD card, finished ATSAM3X
Parts:
- added C? (x2): 100n, symbol Device:C
- added C?: 10n, symbol Device:C
- added C? (x4): 22p, symbol Device:C
- added C?: 22p, symbol Device:C_Small
- added D?: Green, symbol Device:LED
- added FB?: MH2029-300Y, symbol Device:Ferrite_Bead
- added J?: Micro_SD_Card, symbol Connector:Micro_SD_Card
- added R? (x2): 39R 1%, symbol Device:R_Small
- added R?: 6.8k 1%, symbol Device:R_Small
- added R?: 100k, symbol Device:R_Small
- added R?: 1k, symbol Device:R
- added SW?: SW_DPDT_x2, symbol Switch:SW_DPDT_x2
- added SW?: SW_MEC_5G, symbol Switch:SW_MEC_5G
- added Y?: 12MHz KX-7 20pF, symbol Device:Crystal_GND24_Small
- added Y?: 32.768kHz, symbol Device:Crystal_Small
- F?: value Polyfuse -> MF-MSMF050-2 500mA
Connections:
- net +3V3: now also C?.2, C?.2, FB?.2, J?.4 (VDD), R?.1, R?.2
- net -5V: now also U?.4 (V-)
- net 9V_RAW: now also SW?.2 (B); no longer FB?.2
- net AD0: now also U?.78 (PA16)
- net AD1: now also U?.79 (PA24)
- net D+: now also U?.37 (DHSDP), R?.1
- net D-: now also U?.38 (DHSDM), R?.1
- net DAC0: now also U?.76 (PB15)
- net DAC1: now also U?.77 (PB16)
- net GND: now also C?.1, J?.R, J?.T, R?.1, U?.46 (JTAGSEL), U?.51 (TST), C?.1, C?.1, C?.1, C?.1, C?.1, C?.1, C?.2, D?.1 (K), J?.6 (VSS), R?.1, SW?.1 (A), SW?.2 (A), Y?.2, Y?.4
- net UOTGID: now also U?.129 (PB11)
- net VBUS: now also U?.39 (VBUS)
- net PIN22: now reaches U?.1 (PB26)
- net PIN45: now reaches U?.100 (PC18)
- net PIN44: now reaches U?.101 (PC19)
- net PWM10: now reaches U?.102 (PC29)
- net RXI: now reaches U?.103 (PC30)
- net TXL: now reaches U?.107 (PA21)
- net MISO: now reaches U?.108 (PA25)
- net MISO: now also J?.7 (DAT0)
- net MOSI: now reaches U?.109 (PA26)
- net MOSI: now also J?.3 (CMD)
- net SPCK: now reaches U?.110 (PA27)
- net SPCK: now also J?.5 (CLK)
- net SS0PWM10: now reaches U?.111 (PA28)
- net SS1PWM4: now reaches U?.112 (PA29)
- net ETX_CLK: now reaches U?.113 (PB0)
- net ETX_EN: now reaches U?.114 (PB1)
- net ETXD0: now reaches U?.115 (PB2)
- net PIN36: now reaches U?.116 (PC4)
- net ETXD1: now reaches U?.118 (PB3)
- net ERX_DV: now reaches U?.119 (PB4)
- net ERXD0: now reaches U?.120 (PB5)
- net ERXD1: now reaches U?.121 (PB6)
- net ERX_ER: now reaches U?.122 (PB7)
- net EMDC: now reaches U?.123 (PB8)
- net EMDIO: now reaches U?.127 (PB9)
- net UOTGVBOF: now reaches U?.128 (PB10)
- net PIN25: now reaches U?.13 (PD0)
- net PWM9: now reaches U?.132 (PC21)
- net PWM8: now reaches U?.133 (PC22)
- net PWM7: now reaches U?.134 (PC23)
- net PWM6: now reaches U?.135 (PC24)
- net PWM5: now reaches U?.136 (PC25)
- net PWM4: now reaches U?.137 (PC26)
- net PWM3: now reaches U?.139 (PC28)
- net PIN26: now reaches U?.14 (PD1)
- net CANTX1IO: now reaches U?.140 (PB14)
- net SS3: now reaches U?.142 (PB23)
- net PWM2: now reaches U?.144 (PB25)
- net PIN27: now reaches U?.15 (PD2)
- net PIN28: now reaches U?.16 (PD3)
- net TXD0: now reaches U?.17 (PD4)
- net RXD0: now reaches U?.18 (PD5)
- net PIN29: now reaches U?.19 (PD6)
- net TX: now reaches U?.2 (PA9)
- net PWM11: now reaches U?.20 (PD7)
- net PWM12: now reaches U?.21 (PD8)
- net PIN30: now reaches U?.22 (PD9)
- net CANTX0: now reaches U?.23 (PA0)
- net CANRX0: now reaches U?.24 (PA1)
- net EEXTINT: now reaches U?.25 (PA5)
- net PIN31: now reaches U?.26 (PA7)
- net RX: now reaches U?.27 (PA8)
- net JTAG_TCK: now reaches U?.28 (PB28)
- net JTAG_TDI: now reaches U?.29 (PB29)
- net RXD2: now reaches U?.3 (PA10)
- net JTAG_TDO: now reaches U?.30 (PB30)
- net JTAG_TMS: now reaches U?.31 (PB31)
- net PIN32: now reaches U?.32 (PD10)
- net XOUT: now reaches U?.35 (XOUT)
- net XOUT: now also C?.2, Y?.1
- net XIN: now reaches U?.36 (XIN)
- net XIN: now also C?.2, Y?.3
- net TXD2: now reaches U?.4 (PA11)
- net at U?.40 (VBG): now also C?.1, R?.2
- net at U?.42 (DFSDP): now also R?.2
- net at U?.43 (DFSDM): now also R?.2
- net MASTER_RESET: now reaches U?.47 (NRSTB)
- net MASTER_RESET: now also C?.1, SW?.3 (B), SW?.4 (B)
- net XIN32: now reaches U?.48 (XIN32)
- net XIN32: now also C?.2, Y?.1
- net XOUT32: now reaches U?.49 (XOUT32)
- net XOUT32: now also C?.2, Y?.2
- net RXD1: now reaches U?.5 (PA12)
- net at U?.53 (FWUP): now also R?.1
- net PIN33: now reaches U?.55 (PC1)
- net PIN34: now reaches U?.59 (PC2)
- net TXD1: now reaches U?.6 (PA13)
- net PIN35: now reaches U?.60 (PC3)
- net PIN37: now reaches U?.63 (PC5)
- net PIN38: now reaches U?.64 (PC6)
- net PIN39: now reaches U?.65 (PC7)
- net PIN40: now reaches U?.66 (PC8)
- net PIN41: now reaches U?.67 (PC9)
- net PWM13: now reaches U?.68 (PB27)
- net PIN23: now reaches U?.7 (PA14)
- net SCL1: now reaches U?.70 (PA18)
- net PIN42: now reaches U?.71 (PA19)
- net PIN43: now reaches U?.72 (PA20)
- net at U?.75 (ADVREF): now also C?.2, FB?.1
- net PIN24: now reaches U?.8 (PA15)
- net AD2: now reaches U?.80 (PA23)
- net AD3: now reaches U?.81 (PA22)
- net AD4: now reaches U?.82 (PA6)
- net AD5: now reaches U?.83 (PA4)
- net AD6: now reaches U?.84 (PA3)
- net AD7: now reaches U?.85 (PA2)
- net SDA0-3: now reaches U?.86 (PB12)
- net SCL0-3: now reaches U?.87 (PB13)
- net AD8: now reaches U?.88 (PB17)
- net AD9: now reaches U?.89 (PB18)
- net SDA1: now reaches U?.9 (PA17)
- net AD10: now reaches U?.90 (PB19)
- net AD11: now reaches U?.91 (PB20)
- net AD14: now reaches U?.92 (PB21)
- net PIN51: now reaches U?.94 (PC12)
- net PIN50: now reaches U?.95 (PC13)
- net PIN49: now reaches U?.96 (PC14)
- net PIN48: now reaches U?.97 (PC15)
- net PIN47: now reaches U?.98 (PC16)
- net PIN46: now reaches U?.99 (PC17)
- new net: FB?.2, SW?.1 (A)
- new net: D?.2 (A), R?.2
- new net CS: J?.2 (DAT3/CD)
- no-connect marks 3 -> 14
Other:
- moved on the sheet: C?, D?, F?, FB?, J?, JP?, R?, RV?, U?, U?A, U?B

Commit message: Added images of schematic and test files
Parts:
- removed C?: CP1, symbol Device:CP1
- removed R? (x2): 10M, symbol Device:R
- removed U?: TL072, symbol Regulator_SwitchedCapacitor:LTC1044
- added SW?: Rotary_Encoder_Switch, symbol Device:Rotary_Encoder_Switch
- added U?: LTC1044, symbol Regulator_SwitchedCapacitor:LTC1044
- J?: symbol Connector:USB_OTG -> DueFinn-rescue:USB_OTG-Connector
- R?: value ??? -> 10k
Connections:
- net +5V: now also U?.1 (BOOST), U?.8 (V+)
- net -5V: now also U?.5 (VOUT)
- net GND: now also U?.3 (GND); no longer J?.R
- net at C?.1: now also U?.2 (CAP+)
- net at C?.2: now also U?.4 (CAP-)
- net at C?.2, R?.2, U?.7: now also J?.R, J?.S
Other:
- note removed: "?"
- moved on the sheet: C?, D?, L?, R?, U?
